File: CAN_BDC.sch (KiCad schematic (older format))
At the start: 26 parts, among them P1 CONN_01X05, P2 CONN_01X02, P3 CONN_01X02, P4 CONN_01X04, P5 CONN_01X02, U1 STM32F042C6Ux, U2 PSD2CAN, U3 SN65HVD232D, U4 drv8850, U5 MCP1700T-3302E/TT

Commit message: Footpritns addition.
Footpritns addition.
Parts:
- C1, C10, C2, C3, C4, C5, C8, C9: footprint Resistors_SMD:R_0805 -> Capacitors_SMD:C_0402
- C6: footprint Resistors_SMD:R_0805 -> Capacitors_SMD:C_0805
- C7: value 0.1u -> 2.2u; footprint Resistors_SMD:R_0805 -> Capacitors_SMD:C_0402
- R2, R4, R5: footprint Resistors_SMD:R_0805 -> Resistors_SMD:R_0402
- R3: footprint Resistors_SMD:R_0603 -> Resistors_SMD:R_0402
- R6: value 3k -> 3k/127k; footprint Resistors_SMD:R_0805 -> Resistors_SMD:R_0402
- R7: value 1k -> 1k/40.2k; footprint Resistors_SMD:R_0805 -> Resistors_SMD:R_0402
Connections:
- wire segments 50 -> 51
Changed lines of the file:
@@
 F 0 "R3" H 1980 1154 50  0000 R CNN
 F 1 "10k" H 1980 1245 50  0000 R CNN
-F 2 "Resistors_SMD:R_0603" H 1980 1291 50  0001 R CNN
+F 2 "Resistors_SMD:R_0402" H 1980 1291 50  0001 R CNN
 F 3 "" H 2050 1200 50  0000 C CNN
 	1    2050 1200
@@
 F 0 "C4" H 9065 1046 50  0000 L CNN
 F 1 "10nC" H 9065 955 50  0000 L CNN
-F 2 "Resistors_SMD:R_0805" H 8988 850 50  0001 C CNN
+F 2 "Capacitors_SMD:C_0402" H 8988 850 50  0001 C CNN
 F 3 "" H 8950 1000 50  0000 C CNN
 	1    8950 1000
@@
 F 0 "C5" H 9465 1046 50  0000 L CNN
 F 1 "100nC" H 9465 955 50  0000 L CNN
-F 2 "Resistors_SMD:R_0805" H 9388 850 50  0001 C CNN
+F 2 "Capacitors_SMD:C_0402" H 9388 850 50  0001 C CNN
 F 3 "" H 9350 1000 50  0000 C CNN
 	1    9350 1000
@@
 F 0 "C3" H 10600 5200 50  0000 L CNN
 F 1 "10u" H 10650 5100 50  0000 L CNN
-F 2 "Resistors_SMD:R_0805" H 10838 5050 50  0001 C CNN
+F 2 "Capacitors_SMD:C_0402" H 10838 5050 50  0001 C CNN
 F 3 "" H 10800 5200 50  0000 C CNN
 	1    10800 5200
@@
 F 0 "C2" H 10300 5200 50  0000 L CNN
 F 1 "100n" H 10300 5100 50  0000 L CNN
-F 2 "Resistors_SMD:R_0805" H 10538 5050 50  0001 C CNN
+F 2 "Capacitors_SMD:C_0402" H 10538 5050 50  0001 C CNN
 F 3 "" H 10500 5200 50  0000 C CNN
 	1    10500 5200
@@
 $EndComp
 $Comp
-L C C1
-U 1 1 57F80A8D
-P 3100 6300
-F 0 "C1" V 3050 6100 50  0000 L CNN
-F 1 "0.1u" V 3150 6100 50  0000 L CNN
-F 2 "Resistors_SMD:R_0805" H 3138 6150 50  0001 C CNN
-F 3 "" H 3100 6300 50  0000 C CNN
-	1    3100 6300
-	0    1    1    0
-$EndComp
-$Comp
-L C C6
-U 1 1 57F80CC3
-P 3600 6250
-F 0 "C6" H 3715 6296 50  0000 L CNN
-F 1 "10u" H 3715 6205 50  0000 L CNN
-F 2 "Resistors_SMD:R_0805" H 3638 6100 50  0001 C CNN
-F 3 "" H 3600 6250 50  0000 C CNN
-	1    3600 6250
-	-1   0    0    1
-$EndComp
-$Comp
 L C C8
 U 1 1 57F80D21
@@
 F 0 "C8" H 4165 6296 50  0000 L CNN
 F 1 "0.1u" H 4165 6205 50  0000 L CNN
-F 2 "Resistors_SMD:R_0805" H 4088 6100 50  0001 C CNN
+F 2 "Capacitors_SMD:C_0402" H 4088 6100 50  0001 C CNN
 F 3 "" H 4050 6250 50  0000 C CNN
 	1    4050 6250
@@
 U 1 1 57F81C61
 P 3250 6400
-F 0 "R5" V 3150 6550 50  0000 R CNN
+F 0 "R5" V 3250 6450 50  0000 R CNN
 F 1 "4.3k" V 3150 6450 50  0000 R CNN
-F 2 "Resistors_SMD:R_0805" H 3180 6491 50  0001 R CNN
+F 2 "Resistors_SMD:R_0402" H 3180 6491 50  0001 R CNN
 F 3 "" H 3250 6400 50  0000 C CNN
 	1    3250 6400
 	0    -1   -1   0
-$EndComp
-$Comp
-L GNDA #PWR022
-U 1 1 57F820AC
-P 3400 6400
-F 0 "#PWR022" H 3400 6150 50  0001 C CNN
-F 1 "GNDA" H 3450 6250 50  0000 C CNN
-F 2 "" H 3400 6400 50  0000 C CNN
-F 3 "" H 3400 6400 50  0000 C CNN
-	1    3400 6400
-	1    0    0    -1
 $EndComp
 $Comp
@@
 U 1 1 57F83B1D
 P 1400 6600
-F 0 "R4" V 1300 6750 50  0000 R CNN
-F 1 "24k" V 1300 6650 50  0000 R CNN
-F 2 "Resistors_SMD:R_0805" H 1330 6691 50  0001 R CNN
+F 0 "R4" V 1400 6650 50  0000 R CNN
+F 1 "24k" V 1300 6700 50  0000 R CNN
+F 2 "Resistors_SMD:R_0402" H 1330 6691 50  0001 R CNN
 F 3 "" H 1400 6600 50  0000 C CNN
 	1    1400 6600
@@
 $EndComp
 $Comp
-L GNDA #PWR023
+L GNDA #PWR022
 U 1 1 57F83C95
 P 1250 6850
-F 0 "#PWR023" H 1250 6600 50  0001 C CNN
+F 0 "#PWR022" H 1250 6600 50  0001 C CNN
 F 1 "GNDA" H 1258 6677 50  0000 C CNN
 F 2 "" H 1250 6850 50  0000 C CNN
@@
 F 0 "R2" V 800 6400 50  0000 R CNN
 F 1 "0" V 800 6300 50  0000 R CNN
-F 2 "Resistors_SMD:R_0805" H 830 6391 50  0001 R CNN
+F 2 "Resistors_SMD:R_0402" H 830 6391 50  0001 R CNN
 F 3 "" H 900 6300 50  0000 C CNN
 	1    900  6300
@@
 $EndComp
 $Comp
-L +5V #PWR024
+L +5V #PWR023
 U 1 1 57F843CB
 P 4050 6100
-F 0 "#PWR024" H 4050 5950 50  0001 C CNN
+F 0 "#PWR023" H 4050 5950 50  0001 C CNN
 F 1 "+5V" H 4068 6273 50  0000 C CNN
 F 2 "" H 4050 6100 50  0000 C CNN
@@
 $EndComp
 $Comp
-L +5V #PWR025
+L +5V #PWR024
 U 1 1 57F84552
 P 900 6150
-F 0 "#PWR025" H 900 6000 50  0001 C CNN
+F 0 "#PWR024" H 900 6000 50  0001 C CNN
 F 1 "+5V" H 918 6323 50  0000 C CNN
 F 2 "" H 900 6150 50  0000 C CNN
@@
 P 3400 7000
 F 0 "R6" H 3350 7000 50  0000 R CNN
-F 1 "3k" H 3550 7000 50  0000 R CNN
-F 2 "Resistors_SMD:R_0805" H 3330 7091 50  0001 R CNN
+F 1 "3k/127k" H 3300 6900 50  0000 R CNN
+F 2 "Resistors_SMD:R_0402" H 3330 7091 50  0001 R CNN
 F 3 "" H 3400 7000 50  0000 C CNN
 	1    3400 7000
@@
 U 1 1 57F85142
 P 3400 7300
-F 0 "R7" H 3350 7300 50  0000 R CNN
-F 1 "1k" H 3550 7300 50  0000 R CNN
-F 2 "Resistors_SMD:R_0805" H 3330 7391 50  0001 R CNN
+F 0 "R7" H 3350 7250 50  0000 R CNN
+F 1 "1k/40.2k" H 3350 7150 50  0000 R CNN
+F 2 "Resistors_SMD:R_0402" H 3330 7391 50  0001 R CNN
 F 3 "" H 3400 7300 50  0000 C CNN
 	1    3400 7300
@@
 $EndComp
 $Comp
-L GNDA #PWR026
+L GNDA #PWR025
 U 1 1 57F85873
 P 3700 7500
-F 0 "#PWR026" H 3700 7250 50  0001 C CNN
+F 0 "#PWR025" H 3700 7250 50  0001 C CNN
 F 1 "GNDA" H 3708 7327 50  0000 C CNN
 F 2 "" H 3700 7500 50  0000 C CNN
@@
 $EndComp
 $Comp
-L +3.3V #PWR027
+L +3.3V #PWR026
 U 1 1 57F859A8
 P 3700 6850
-F 0 "#PWR027" H 3700 6700 50  0001 C CNN
+F 0 "#PWR026" H 3700 6700 50  0001 C CNN
 F 1 "+3.3V" H 3800 7000 50  0000 C CNN
 F 2 "" H 3700 6850 50  0000 C CNN
@@
 U 1 1 57F86494
 P 3700 7200
-F 0 "C7" H 3700 7100 50  0000 L CNN
-F 1 "0.1u" H 3500 7100 50  0000 L CNN
-F 2 "Resistors_SMD:R_0805" H 3738 7050 50  0001 C CNN
+F 0 "C7" H 3500 7150 50  0000 L CNN
+F 1 "2.2u" H 3400 7250 50  0000 L CNN
+F 2 "Capacitors_SMD:C_0402" H 3738 7050 50  0001 C CNN
 F 3 "" H 3700 7200 50  0000 C CNN
 	1    3700 7200
@@
 $EndComp
 $Comp
-L GND #PWR028
+L GND #PWR027
 U 1 1 57F9604D
 P 5750 5600
-F 0 "#PWR028" H 5750 5350 50  0001 C CNN
+F 0 "#PWR027" H 5750 5350 50  0001 C CNN
 F 1 "GND" H 5758 5427 50  0000 C CNN
 F 2 "" H 5750 5600 50  0000 C CNN
@@
 F 0 "C9" H 5065 5496 50  0000 L CNN
 F 1 "1u" H 5065 5405 50  0000 L CNN
-F 2 "Resistors_SMD:R_0805" H 4988 5300 50  0001 C CNN
+F 2 "Capacitors_SMD:C_0402" H 4988 5300 50  0001 C CNN
 F 3 "" H 4950 5450 50  0000 C CNN
 	1    4950 5450
@@
 F 0 "C10" H 5550 5450 50  0000 L CNN
 F 1 "1u" H 5550 5350 50  0000 L CNN
-F 2 "Resistors_SMD:R_0805" H 5788 5300 50  0001 C CNN
+F 2 "Capacitors_SMD:C_0402" H 5788 5300 50  0001 C CNN
 F 3 "" H 5750 5450 50  0000 C CNN
 	1    5750 5450
 	-1   0    0    1
+$EndComp
+$Comp
+L +5V #PWR028
+U 1 1 57F969C6
+P 4950 5300
+F 0 "#PWR028" H 4950 5150 50  0001 C CNN
+F 1 "+5V" H 4968 5473 50  0000 C CNN
+F 2 "" H 4950 5300 50  0000 C CNN
+F 3 "" H 4950 5300 50  0000 C CNN
+	1    4950 5300
+	1    0    0    -1
+$EndComp
+$Comp
+L +3.3V #PWR029
+U 1 1 57F96BE3
+P 5750 5300
+F 0 "#PWR029" H 5750 5150 50  0001 C CNN
+F 1 "+3.3V" H 5850 5450 50  0000 C CNN
+F 2 "" H 5750 5300 50  0000 C CNN
+F 3 "" H 5750 5300 50  0000 C CNN
+	1    5750 5300
+	1    0    0    -1
+$EndComp
+Text GLabel 2900 5050 1    60   Input ~ 0
+BMF2
+Text GLabel 1550 5050 1    60   Input ~ 0
+BMF1
+$Comp
+L GNDA #PWR030
+U 1 1 57F9B056
+P 4950 5600
+F 0 "#PWR030" H 4950 5350 50  0001 C CNN
+F 1 "GNDA" H 4958 5427 50  0000 C CNN
+F 2 "" H 4950 5600 50  0000 C CNN
+F 3 "" H 4950 5600 50  0000 C CNN
+	1    4950 5600
+	1    0    0    -1
+$EndComp
+$Comp
+L C C6
+U 1 1 57F80CC3
+P 3600 6250
+F 0 "C6" H 3715 6296 50  0000 L CNN
+F 1 "10u" H 3715 6205 50  0000 L CNN
+F 2 "Capacitors_SMD:C_0805" H 3638 6100 50  0001 C CNN
+F 3 "" H 3600 6250 50  0000 C CNN
+	1    3600 6250
+	-1   0    0    1
+$EndComp
+$Comp
+L GNDA #PWR031
+U 1 1 57F820AC
+P 3400 6400
+F 0 "#PWR031" H 3400 6150 50  0001 C CNN
+F 1 "GNDA" H 3450 6250 50  0000 C CNN
+F 2 "" H 3400 6400 50  0000 C CNN
+F 3 "" H 3400 6400 50  0000 C CNN
+	1    3400 6400
+	1    0    0    -1
 $EndComp
 Wire Wire Line
@@
 Wire Wire Line
 	2900 6400 3100 6400
-Wire Wire Line
-	2900 6300 2950 6300
-Wire Wire Line
-	3250 6000 3250 6300
 Connection ~ 1550 5800
 Connection ~ 1550 5700
@@
 	4950 5600 5750 5600
 Connection ~ 5750 5600
-$Comp
-L +5V #PWR029
-U 1 1 57F969C6
-P 4950 5300
-F 0 "#PWR029" H 4950 5150 50  0001 C CNN
-F 1 "+5V" H 4968 5473 50  0000 C CNN
-F 2 "" H 4950 5300 50  0000 C CNN
-F 3 "" H 4950 5300 50  0000 C CNN
-	1    4950 5300
-	1    0    0    -1
-$EndComp
-$Comp
-L +3.3V #PWR030
-U 1 1 57F96BE3
-P 5750 5300
-F 0 "#PWR030" H 5750 5150 50  0001 C CNN
-F 1 "+3.3V" H 5850 5450 50  0000 C CNN
-F 2 "" H 5750 5300 50  0000 C CNN
-F 3 "" H 5750 5300 50  0000 C CNN
-	1    5750 5300
-	1    0    0    -1
-$EndComp
 Connection ~ 4950 5300
 Connection ~ 5750 5300
 Connection ~ 5350 5600
 Connection ~ 4050 6100
-Text GLabel 2900 5050 1    60   Input ~ 0
-BMF2
 Connection ~ 2900 5150
-Text GLabel 1550 5050 1    60   Input ~ 0
-BMF1
 Connection ~ 1550 5150
-$Comp
-L GNDA #PWR031
-U 1 1 57F9B056
-P 4950 5600
-F 0 "#PWR031" H 4950 5350 50  0001 C CNN
-F 1 "GNDA" H 4958 5427 50  0000 C CNN
-F 2 "" H 4950 5600 50  0000 C CNN
-F 3 "" H 4950 5600 50  0000 C CNN
-	1    4950 5600
-	1    0    0    -1
-$EndComp
 Connection ~ 4950 5600
+Wire Wire Line
+	2900 6300 2950 6300
+Wire Wire Line
+	3250 6000 3250 6300
+$Comp
+L C C1
+U 1 1 57F80A8D
+P 3100 6300
+F 0 "C1" V 3050 6100 50  0000 L CNN
+F 1 "0.1u" V 3150 6100 50  0000 L CNN
+F 2 "Capacitors_SMD:C_0402" H 3138 6150 50  0001 C CNN
+F 3 "" H 3100 6300 50  0000 C CNN
+	1    3100 6300
+	0    1    1    0
+$EndComp
+$Comp
+L GNDA #PWR032
+U 1 1 57FC2643
+P 3850 5600
+F 0 "#PWR032" H 3850 5350 50  0001 C CNN
+F 1 "GNDA" H 3950 5450 50  0000 C CNN
+F 2 "" H 3850 5600 50  0000 C CNN
+F 3 "" H 3850 5600 50  0000 C CNN
+	1    3850 5600
+	1    0    0    -1
+$EndComp
+$Comp
+L GND #PWR033
+U 1 1 57FC269C
+P 3650 5600
+F 0 "#PWR033" H 3650 5350 50  0001 C CNN
+F 1 "GND" H 3658 5427 50  0000 C CNN
+F 2 "" H 3650 5600 50  0000 C CNN
+F 3 "" H 3650 5600 50  0000 C CNN
+	1    3650 5600
+	1    0    0    -1
+$EndComp
+Wire Wire Line
+	3650 5600 3850 5600
 $EndSCHEMATC

Commit message: Layout Creation
Layout Creation
Parts:
- removed C7: 2.2u, Capacitors_SMD:C_0402, symbol C
- removed R2: 0, Resistors_SMD:R_0402, symbol R
- removed R6: 3k/127k, Resistors_SMD:R_0402, symbol R
- removed R7: 1k/40.2k, Resistors_SMD:R_0402, symbol R
- added C11: 0.1u, Capacitors_SMD:c_elec_3x5.3, symbol C
Connections:
- net labels added: nSLEEP
- wire segments 51 -> 41
Other:
- moved on the sheet: C10
Changed lines of the file:
@@
-$EndComp
-$Comp
-L R R2
-U 1 1 57F83D29
-P 900 6300
-F 0 "R2" V 800 6400 50  0000 R CNN
-F 1 "0" V 800 6300 50  0000 R CNN
-F 2 "Resistors_SMD:R_0402" H 830 6391 50  0001 R CNN
-F 3 "" H 900 6300 50  0000 C CNN
-	1    900  6300
-	1    0    0    -1
 $EndComp
 $Comp
@@
 	1    0    0    -1
 $EndComp
-$Comp
-L +5V #PWR024
-U 1 1 57F84552
-P 900 6150
-F 0 "#PWR024" H 900 6000 50  0001 C CNN
-F 1 "+5V" H 918 6323 50  0000 C CNN
-F 2 "" H 900 6150 50  0000 C CNN
-F 3 "" H 900 6150 50  0000 C CNN
-	1    900  6150
-	1    0    0    -1
-$EndComp
-$Comp
-L R R6
-U 1 1 57F84FFF
-P 3400 7000
-F 0 "R6" H 3350 7000 50  0000 R CNN
-F 1 "3k/127k" H 3300 6900 50  0000 R CNN
-F 2 "Resistors_SMD:R_0402" H 3330 7091 50  0001 R CNN
-F 3 "" H 3400 7000 50  0000 C CNN
-	1    3400 7000
-	1    0    0    -1
-$EndComp
-$Comp
-L R R7
-U 1 1 57F85142
-P 3400 7300
-F 0 "R7" H 3350 7250 50  0000 R CNN
-F 1 "1k/40.2k" H 3350 7150 50  0000 R CNN
-F 2 "Resistors_SMD:R_0402" H 3330 7391 50  0001 R CNN
-F 3 "" H 3400 7300 50  0000 C CNN
-	1    3400 7300
-	1    0    0    -1
-$EndComp
-$Comp
-L GNDA #PWR025
-U 1 1 57F85873
-P 3700 7500
-F 0 "#PWR025" H 3700 7250 50  0001 C CNN
-F 1 "GNDA" H 3708 7327 50  0000 C CNN
-F 2 "" H 3700 7500 50  0000 C CNN
-F 3 "" H 3700 7500 50  0000 C CNN
-	1    3700 7500
-	1    0    0    -1
-$EndComp
-$Comp
-L +3.3V #PWR026
-U 1 1 57F859A8
-P 3700 6850
-F 0 "#PWR026" H 3700 6700 50  0001 C CNN
-F 1 "+3.3V" H 3800 7000 50  0000 C CNN
-F 2 "" H 3700 6850 50  0000 C CNN
-F 3 "" H 3700 6850 50  0000 C CNN
-	1    3700 6850
-	1    0    0    -1
-$EndComp
-$Comp
-L C C7
-U 1 1 57F86494
-P 3700 7200
-F 0 "C7" H 3500 7150 50  0000 L CNN
-F 1 "2.2u" H 3400 7250 50  0000 L CNN
-F 2 "Capacitors_SMD:C_0402" H 3738 7050 50  0001 C CNN
-F 3 "" H 3700 7200 50  0000 C CNN
-	1    3700 7200
-	-1   0    0    1
-$EndComp
 Text Notes 700  4650 0    118  ~ 0
 MOTOR DRIVE
@@
 L GND #PWR027
 U 1 1 57F9604D
-P 5750 5600
-F 0 "#PWR027" H 5750 5350 50  0001 C CNN
-F 1 "GND" H 5758 5427 50  0000 C CNN
-F 2 "" H 5750 5600 50  0000 C CNN
-F 3 "" H 5750 5600 50  0000 C CNN
-	1    5750 5600
+P 5850 5600
+F 0 "#PWR027" H 5850 5350 50  0001 C CNN
+F 1 "GND" H 5858 5427 50  0000 C CNN
+F 2 "" H 5850 5600 50  0000 C CNN
+F 3 "" H 5850 5600 50  0000 C CNN
+	1    5850 5600
 	1    0    0    -1
 $EndComp
@@
 L C C10
 U 1 1 57F96647
-P 5750 5450
-F 0 "C10" H 5550 5450 50  0000 L CNN
-F 1 "1u" H 5550 5350 50  0000 L CNN
-F 2 "Capacitors_SMD:C_0402" H 5788 5300 50  0001 C CNN
-F 3 "" H 5750 5450 50  0000 C CNN
-	1    5750 5450
+P 5850 5450
+F 0 "C10" H 5950 5500 50  0000 L CNN
+F 1 "1u" H 6000 5400 50  0000 L CNN
+F 2 "Capacitors_SMD:C_0402" H 5888 5300 50  0001 C CNN
+F 3 "" H 5850 5450 50  0000 C CNN
+	1    5850 5450
 	-1   0    0    1
 $EndComp
@@
 L +3.3V #PWR029
 U 1 1 57F96BE3
-P 5750 5300
-F 0 "#PWR029" H 5750 5150 50  0001 C CNN
-F 1 "+3.3V" H 5850 5450 50  0000 C CNN
-F 2 "" H 5750 5300 50  0000 C CNN
-F 3 "" H 5750 5300 50  0000 C CNN
-	1    5750 5300
+P 5850 5300
+F 0 "#PWR029" H 5850 5150 50  0001 C CNN
+F 1 "+3.3V" H 5950 5450 50  0000 C CNN
+F 2 "" H 5850 5300 50  0000 C CNN
+F 3 "" H 5850 5300 50  0000 C CNN
+	1    5850 5300
 	1    0    0    -1
 $EndComp
@@
 	2900 6000 3250 6000
 Wire Wire Line
-	2900 6100 4050 6100
+	2900 6100 4450 6100
 Wire Wire Line
 	2900 6200 3250 6200
@@
 Connection ~ 3600 6400
 Wire Wire Line
-	4050 6400 3600 6400
+	3600 6400 4450 6400
 Wire Wire Line
 	2450 5350 2450 5400
@@
 Connection ~ 2900 5700
 Wire Wire Line
-	1550 6500 900  6500
-Wire Wire Line
-	900  6500 900  6450
-Wire Wire Line
 	1250 6600 1250 6850
 Wire Wire Line
-	2900 6500 3050 6500
-Wire Wire Line
-	3050 6500 3050 6850
-Wire Wire Line
-	3050 6850 3700 6850
-Wire Wire Line
-	2900 6600 2900 7150
-Wire Wire Line
-	2900 7150 3400 7150
-Connection ~ 3400 7150
-Connection ~ 3400 6850
-Wire Wire Line
-	3700 6850 3700 7050
-Wire Wire Line
-	3700 7500 3400 7500
-Wire Wire Line
-	3400 7500 3400 7450
-Wire Wire Line
-	3700 7500 3700 7350
-Connection ~ 3700 7500
-Connection ~ 3700 6850
-Wire Wire Line
 	1550 5050 1550 5900
 Wire Wire Line
@@
 	2900 5050 2900 5900
 Wire Wire Line
-	4950 5600 5750 5600
-Connection ~ 5750 5600
+	4950 5600 5850 5600
+Connection ~ 5850 5600
 Connection ~ 4950 5300
-Connection ~ 5750 5300
+Connection ~ 5850 5300
 Connection ~ 5350 5600
 Connection ~ 4050 6100
@@
 Wire Wire Line
 	3650 5600 3850 5600
+$Comp
+L C C11
+U 1 1 57FBD962
+P 4450 6250
+F 0 "C11" H 4565 6296 50  0000 L CNN
+F 1 "0.1u" H 4550 6200 50  0000 L CNN
+F 2 "Capacitors_SMD:c_elec_3x5.3" H 4488 6100 50  0001 C CNN
+F 3 "" H 4450 6250 50  0000 C CNN
+	1    4450 6250
+	-1   0    0    1
+$EndComp
+Connection ~ 4050 6400
+Wire Wire Line
+	5750 5300 5850 5300
+Text GLabel 1550 6400 0    60   Input ~ 0
+nSLEEP
 $EndSCHEMATC
