File: CAN_BDC.kicad_pcb (KiCad board)
At the start: 2 copper layers, 26 x 28.5 mm, 35 parts, among them P1 CONN_01X02, P2 CONN_01X05, P3 CONN_01X02, P4 CONN_01X02, P5 CONN_01X02, P6 CONN_01X02, P7 CONN_01X04, P8 CONN_01X01, P9 CONN_01X02, U1 PSD2CAN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

Commit message: Footprint update.
Parts:
- moved R6 7.36 mm to (153.0, 87.2), turned to 180 degrees
- moved R2 5.08 mm to (151.0, 89.0), turned to 270 degrees
- moved U5 0.95 mm to (147.2, 88.0)
- moved R1 0.50 mm to (143.1, 88.0)
- moved P1 0.41 mm to (141.6, 85.7)
- moved C5 0.36 mm to (151.2, 98.7)
Routing:
- net Net-(R2-Pad2): track 2.91 -> 11.7 mm
- net Net-(R1-Pad1): track 4.91 -> 6.37 mm
- net Net-(C5-Pad1): track 10.2 -> 11.3 mm
- net Net-(D1-Pad1): track 8.84 -> 9.82 mm
Changed lines of the file:
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@@
   (general
     (links 87)
-    (no_connects 20)
-    (area 137.075 82.125 165.304762 113.7393)
+    (no_connects 32)
+    (area 137.075 82.916667 165.304762 113.7393)
     (thickness 1.6)
     (drawings 8)
-    (tracks 232)
+    (tracks 244)
     (zones 0)
     (modules 35)
@@
   (page A4)
   (layers
-    (0 F.Cu signal)
+    (0 F.Cu signal hide)
     (31 B.Cu signal)
     (32 B.Adhes user)
     (33 F.Adhes user)
     (34 B.Paste user)
-    (35 F.Paste user)
+    (35 F.Paste user hide)
     (36 B.SilkS user)
     (37 F.SilkS user)
@@
   )
   (setup
-    (last_trace_width 0.25)
+    (last_trace_width 0.5)
     (user_trace_width 0.5)
     (user_trace_width 0.75)
@@
     (aux_axis_origin 161.4 110.05)
     (grid_origin 161.4 110.05)
-    (visible_elements 7FFFFF7F)
+    (visible_elements 7FFFFD7F)
     (pcbplotparams
       (layerselection 0x3ffff_ffffffff)
@@
   )
   (module Resistors_SMD:R_0603 (layer B.Cu)
-    (at 143.55 88.05)
+    (at 143.05 88.05)
     (descr "Resistor SMD 0603, reflow soldering, Vishay (see dcrcw.pdf)")
     (tags "resistor 0603")
@@
   )
   (module usb_ccb_custom:SOIC-8 (layer B.Cu)
-    (at 147.15 89 180)
+    (at 147.2 88.05 180)
     (fp_text reference U5 (at -0.885 0.31 450) (layer B.SilkS)
       (effects (font (size 0.4 0.4) (thickness 0.09)) (justify mirror))
@@
   )
   (module Pin_Headers:Pin_Header_Straight_1x02_Pitch2.00mm (layer F.Cu)
-    (at 142 85.55 90)
+    (at 141.6 85.65 90)
     (descr "Through hole pin header, 1x02, 2.00mm pitch, single row")
     (tags "pin header single row")
@@
   )
   (module Resistors_SMD:R_0603 (layer B.Cu)
-    (at 148.65 84.55 180)
+    (at 151 89.05 270)
     (descr "Resistor SMD 0603, reflow soldering, Vishay (see dcrcw.pdf)")
     (tags "resistor 0603")
     (attr smd)
-    (fp_text reference R2 (at -1.75 -0.05 270) (layer B.SilkS)
-      (effects (font (size 0.4 0.4) (thickness 0.09)) (justify mirror))
-    )
-    (fp_text value 0.33 (at 0 -1.9 180) (layer B.Fab) hide
+    (fp_text reference R2 (at -0.4 -1.2 450) (layer B.SilkS)
+      (effects (font (size 0.4 0.4) (thickness 0.09)) (justify mirror))
+    )
+    (fp_text value 0.33 (at 0 -1.9 270) (layer B.Fab) hide
       (effects (font (size 0.4 0.4) (thickness 0.09)) (justify mirror))
     )
@@
     (fp_line (start 0.5 -0.675) (end -0.5 -0.675) (layer B.SilkS) (width 0.15))
     (fp_line (start -0.5 0.675) (end 0.5 0.675) (layer B.SilkS) (width 0.15))
-    (pad 1 smd rect (at -0.75 0 180) (size 0.5 0.9) (layers B.Cu B.Paste B.Mask)
+    (pad 1 smd rect (at -0.75 0 270) (size 0.5 0.9) (layers B.Cu B.Paste B.Mask)
       (net 27 "Net-(R2-Pad1)"))
-    (pad 2 smd rect (at 0.75 0 180) (size 0.5 0.9) (layers B.Cu B.Paste B.Mask)
+    (pad 2 smd rect (at 0.75 0 270) (size 0.5 0.9) (layers B.Cu B.Paste B.Mask)
       (net 34 "Net-(R2-Pad2)"))
     (model Resistors_SMD.3dshapes/R_0603.wrl
@@
   )
   (module Capacitors_SMD:C_0805 (layer B.Cu)
-    (at 150.85 98.55 270)
+    (at 151.2 98.65 270)
     (descr "Capacitor SMD 0805, reflow soldering, AVX (see smccp.pdf)")
     (tags "capacitor 0805")
@@
   )
   (module Resistors_SMD:R_0603 (layer B.Cu)
-    (at 146.15 84.55)
+    (at 153 87.25 180)
     (descr "Resistor SMD 0603, reflow soldering, Vishay (see dcrcw.pdf)")
     (tags "resistor 0603")
     (attr smd)
-    (fp_text reference R6 (at -1.55 0 90) (layer B.SilkS)
-      (effects (font (size 0.4 0.4) (thickness 0.09)) (justify mirror))
-    )
-    (fp_text value 0 (at 0 -1.9) (layer B.Fab) hide
+    (fp_text reference R6 (at -1.55 0 270) (layer B.SilkS)
+      (effects (font (size 0.4 0.4) (thickness 0.09)) (justify mirror))
+    )
+    (fp_text value 0 (at 0 -1.9 180) (layer B.Fab) hide
       (effects (font (size 0.4 0.4) (thickness 0.09)) (justify mirror))
     )
@@
     (fp_line (start 0.5 -0.675) (end -0.5 -0.675) (layer B.SilkS) (width 0.15))
     (fp_line (start -0.5 0.675) (end 0.5 0.675) (layer B.SilkS) (width 0.15))
-    (pad 1 smd rect (at -0.75 0) (size 0.5 0.9) (layers B.Cu B.Paste B.Mask)
+    (pad 1 smd rect (at -0.75 0 180) (size 0.5 0.9) (layers B.Cu B.Paste B.Mask)
       (net 11 VPP))
-    (pad 2 smd rect (at 0.75 0) (size 0.5 0.9) (layers B.Cu B.Paste B.Mask)
+    (pad 2 smd rect (at 0.75 0 180) (size 0.5 0.9) (layers B.Cu B.Paste B.Mask)
       (net 34 "Net-(R2-Pad2)"))
     (model Resistors_SMD.3dshapes/R_0603.wrl
@@
   (segment (start 155.039671 102.61) (end 155.629671 103.2) (width 1.5) (layer F.Cu) (net 25))
   (segment (start 153.55 102.61) (end 155.039671 102.61) (width 1.5) (layer F.Cu) (net 25))
-  (segment (start 142.8 88.05) (end 142.8 87.9) (width 0.5) (layer B.Cu) (net 26))
-  (segment (start 142.8 87.9) (end 144.4 86.3) (width 0.5) (layer B.Cu) (net 26))
-  (segment (start 144.4 86.3) (end 145.245 86.3) (width 0.5) (layer B.Cu) (net 26))
-  (segment (start 143.05 89.6) (end 143.05 88.85) (width 0.5) (layer B.Cu) (net 26))
-  (segment (start 142.8 88.6) (end 142.8 88.05) (width 0.5) (layer B.Cu) (net 26))
-  (segment (start 143.05 88.85) (end 142.8 88.6) (width 0.5) (layer B.Cu) (net 26))
-  (segment (start 149.055 86.3) (end 149.055 85.395) (width 0.5) (layer B.Cu) (net 27))
-  (segment (start 149.055 85.395) (end 149.4 85.05) (width 0.5) (layer B.Cu) (net 27))
-  (segment (start 149.4 85.05) (end 149.4 84.55) (width 0.5) (layer B.Cu) (net 27))
-  (segment (start 149.055 86.3) (end 147.785 86.3) (width 0.5) (layer B.Cu) (net 27))
-  (segment (start 149.055 91.7) (end 149.055 86.3) (width 0.5) (layer B.Cu) (net 27))
+  (segment (start 142.3 88.05) (end 142.3 87.85) (width 0.5) (layer B.Cu) (net 26))
+  (segment (start 142.3 87.85) (end 143.374999 86.775001) (width 0.5) (layer B.Cu) (net 26))
+  (segment (start 143.374999 86.775001) (end 144.344999 86.775001) (width 0.5) (layer B.Cu) (net 26))
+  (segment (start 144.344999 86.775001) (end 145.295 85.825) (width 0.5) (layer B.Cu) (net 26))
+  (segment (start 145.295 85.825) (end 145.295 85.35) (width 0.5) (layer B.Cu) (net 26))
+  (segment (start 143.05 89.6) (end 143.05 89) (width 0.5) (layer B.Cu) (net 26))
+  (segment (start 143.05 89) (end 142.3 88.25) (width 0.5) (layer B.Cu) (net 26))
+  (segment (start 142.3 88.25) (end 142.3 88.05) (width 0.5) (layer B.Cu) (net 26))
+  (segment (start 149.105 90.75) (end 149.105 85.845) (width 0.5) (layer B.Cu) (net 27))
+  (segment (start 149.105 85.845) (end 149.105 85.35) (width 0.5) (layer B.Cu) (net 27))
+  (segment (start 151 88.3) (end 149.105 90.195) (width 0.5) (layer B.Cu) (net 27))
+  (segment (start 149.105 90.195) (end 149.105 90.75) (width 0.5) (layer B.Cu) (net 27))
+  (segment (start 147.785 90.8) (end 147.785 91.7) (width 0.5) (layer B.Cu) (net 28) (status 400000))
+  (segment (start 147.785 91.7) (end 147.785 93.5) (width 0.5) (layer B.Cu) (net 28))
+  (segment (start 147.785 90.8) (end 147.835 90.75) (width 0.5) (layer B.Cu) (net 28) (status C00000))
   (segment (start 147.785 93.5) (end 149.4 93.5) (width 0.5) (layer B.Cu) (net 28))
+  (segment (start 149.4 93.5) (end 151.15 91.75) (width 0.5) (layer B.Cu) (net 28))
   (segment (start 151.15 91.75) (end 151.15 91.05) (width 0.5) (layer B.Cu) (net 28))
-  (segment (start 149.4 93.5) (end 151.15 91.75) (width 0.5) (layer B.Cu) (net 28))
   (segment (start 148.4 95.5) (end 148.4 94.5) (width 0.5) (layer B.Cu) (net 28))
   (segment (start 148.4 94.5) (end 147.785 93.885) (width 0.5) (layer B.Cu) (net 28))
   (segment (start 147.785 93.885) (end 147.785 93.5) (width 0.5) (layer B.Cu) (net 28))
-  (segment (start 147.785 93.5) (end 147.785 91.7) (width 0.5) (layer B.Cu) (net 28))
-  (segment (start 146.515 91.7) (end 146.515 97.115) (width 0.5) (layer B.Cu) (net 29))
-  (segment (start 146.9 97.5) (end 151.15 97.5) (width 0.5) (layer B.Cu) (net 29))
+  (segment (start 146.515 91.7) (end 146.515 90.8) (width 0.5) (layer B.Cu) (net 29) (status 800000))
+  (segment (start 146.515 90.8) (end 146.565 90.75) (width 0.5) (layer B.Cu) (net 29) (status C00000))
+  (segment (start 146.515 91.85) (end 146.515 91.7) (width 0.5) (layer B.Cu) (net 29))
   (segment (start 146.515 97.115) (end 146.9 97.5) (width 0.5) (layer B.Cu) (net 29))
+  (segment (start 151.15 97.5) (end 146.9 97.5) (width 0.5) (layer B.Cu) (net 29))
+  (segment (start 146.515 91.85) (end 146.515 97.115) (width 0.5) (layer B.Cu) (net 29))
+  (segment (start 146.515 91.7) (end 146.515 91.85) (width 0.5) (layer B.Cu) (net 29))
   (segment (start 143.2 101.75) (end 143.2 106.5) (width 0.5) (layer B.Cu) (net 30))
   (segment (start 143.2 106.5) (end 142.9 106.8) (width 0.5) (layer B.Cu) (net 30))
@@
   (segment (start 138.348998 103.25) (end 139.767341 103.25) (width 0.25) (layer F.Cu) (net 33))
   (segment (start 141.612649 104.18999) (end 144.291059 106.8684) (width 0.25) (layer F.Cu) (net 33))
-  (segment (start 146.515 86.3) (end 146.515 85.435) (width 0.5) (layer B.Cu) (net 34))
-  (segment (start 146.515 85.435) (end 146.9 85.05) (width 0.5) (layer B.Cu) (net 34))
-  (segment (start 146.9 85.05) (end 146.9 84.55) (width 0.5) (layer B.Cu) (net 34))
-  (segment (start 146.9 84.55) (end 147.9 84.55) (width 0.5) (layer B.Cu) (net 34))
+  (segment (start 152.25 87.25) (end 151.5 87.25) (width 0.5) (layer B.Cu) (net 34))
+  (segment (start 150 84.409998) (end 149.690002 84.1) (width 0.5) (layer B.Cu) (net 34))
+  (segment (start 147.249998 84.1) (end 146.565 84.784998) (width 0.5) (layer B.Cu) (net 34))
+  (segment (start 151.5 87.25) (end 150 85.75) (width 0.5) (layer B.Cu) (net 34))
+  (segment (start 146.565 84.784998) (end 146.565 85.35) (width 0.5) (layer B.Cu) (net 34))
+  (segment (start 150 85.75) (end 150 84.409998) (width 0.5) (layer B.Cu) (net 34))
+  (segment (start 149.690002 84.1) (end 147.249998 84.1) (width 0.5) (layer B.Cu) (net 34))
+  (segment (start 151 89.8) (end 152.25 88.55) (width 0.5) (layer B.Cu) (net 34))
+  (segment (start 152.25 88.55) (end 152.25 87.25) (width 0.5) (layer B.Cu) (net 34))
   (zone (net 2) (net_name GND) (layer F.Cu) (hatch edge 0.508)
     (connect_pads (clearance 0.5))

Commit message: Root full
Root full
Parts:
- L1: footprint usb_ccb_custom:DE0704_Coil -> usb_ccb_custom:DE0704_Coil_2
- L2: footprint Resistors_SMD:R_0805 -> Capacitors_SMD:C_1206
- P1, P3, P4, P5, P6, P7, P9, U3: moved to B.Cu
- P2: footprint usb_ccb_custom:swd_smd_conn5 -> usb_ccb_custom:swd_smd_conn5_x2
- moved P6 26.5 mm to (159.4, 110.3)
- moved C7 23.4 mm to (146.2, 86.0), turned to 180 degrees
- moved R6 22.9 mm to (151.7, 110.2)
- moved L2 22.0 mm to (151.2, 87.2), turned to 90 degrees
- moved R1 21.2 mm to (150.6, 107.8), turned to 270 degrees
- moved R2 20.4 mm to (143.7, 108.2)
- moved P2 19.9 mm to (145.7, 84.3), turned to 270 degrees
- moved P3 19.9 mm to (157.7, 87.0)
- moved U5 19.1 mm to (147.2, 107.2), turned to 0 degrees
- moved R3 16.5 mm to (151.0, 104.8), turned to 90 degrees
- moved C4 15.5 mm to (159.4, 104.3), turned to 270 degrees
- moved D1 13.3 mm to (143.2, 103.2), turned to 90 degrees
- moved P1 11.6 mm to (153.2, 85.0), turned to 270 degrees
- moved C6 10.8 mm to (147.3, 92.2), turned to 180 degrees
- moved P5 9.26 mm to (161.2, 92.3), turned to 0 degrees
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Connections:
- U4 pad 2: DRV_STEP -> DRV_MS1
- U4 pad 23: DRV_nENABLE -> DRV_DIR
- U4 pad 24: DRV_MS1 -> DRV_STEP
- U4 pad 25: DRV_MS2 -> DRV_nSLEEP
- U4 pad 26: DRV_MS3 -> DRV_nRESET
- U4 pad 27: DRV_nRESET -> DRV_MS3
- U4 pad 28: DRV_nSLEEP -> DRV_MS2
- U4 pad 3: DRV_DIR -> DRV_nENABLE
Routing:
- net GND: track 23.7 -> 196.3 mm, vias 3 -> 1
- net CAN_MOD: track 0.57 -> 40.1 mm
- net VPP: track 47.8 -> 14.3 mm, vias 3 -> 0
- net Net-(P2-Pad2): track 14.2 -> 43.4 mm
- net +3V3: track 30.7 -> 58.2 mm, vias 0 -> 3
- net /GPIO4: track 0.00 -> 25.5 mm
- net /GPIO3: track 0.00 -> 24.8 mm
- net /GPIO2: track 0.00 -> 21.0 mm
- net /GPIO1: track 0.00 -> 19.6 mm
- net /USART_RX: track 0.00 -> 18.0 mm
- net /USART_TX: track 0.04 -> 16.5 mm
- net Net-(P8-Pad1): track 17.2 -> 2.82 mm
- net DRV_DIR: track 7.16 -> 18.9 mm
- net DRV_STEP: track 7.26 -> 17.0 mm
- net SW_DIO: track 27.2 -> 18.2 mm
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Other:
- board size 26 x 28.5 mm -> 24 x 28.5 mm
